Commit message: Working velodyne on top of tiago model

File: lcastor_description/robots/tiago-029.urdf.xacro (robot description, xacro)
@@ -27,4 +27,6 @@
     <xacro:arg name="no_safety_eps" default="false"/>
     <xacro:arg name="base_type" default="pmb2"/> <!-- pmb2, omni_base -->
+    <xacro:arg name="organize_cloud" default="true"/>
+    <xacro:arg name="gpu" default="true"/>
     <xacro:property name="wrist_model" value="$(arg wrist_model)" />
     <xacro:property name="end_effector" value="$(arg end_effector)" />
@@ -87,4 +89,6 @@
   <!-- Generic simulator_gazebo plugins -->
   <xacro:include filename="$(find tiago_description)/gazebo/gazebo.urdf.xacro" />
+  <!-- Velodyne VLP-16 -->
+  <xacro:include filename="$(find velodyne_description)/urdf/VLP-16.urdf.xacro"/>
   <!-- Now we can start using the macros included above to define the actual robot -->
   <xacro:if value="${base_type == 'pmb2'}">
@@ -138,5 +142,6 @@
   </link>
   <!-- VLP-16 velodyne -->
-  <xacro:include filename="$(find velodyne_description)/urdf/VLP-16.urdf.xacro" />
-  <xacro:velodyne name="velodyne" parent="torso_lift_link" origin="0 0 0.30 0 0 0"/>
+  <xacro:VLP-16 parent="torso_lift_link" name="velodyne" topic="/velodyne_points" hz="10" gpu="true" >
+    <origin xyz="0 0 0.3" rpy="0 0 0" />
+  </xacro:VLP-16>
 </robot>
